File: hardware/LEC011001.kicad_sch (KiCad schematic)
At the start: 40 parts, among them J1 Button, J2 PWR, J3 CONTACT_1, J4 CONTACT_2, K1 HK19F-5V, Q1 S8050, U1 MC78M05_TO252, U2 NE555D

Commit message: Add prod files
Parts:
- J1, J2: JLCPCB_CORRECTION (none) -> 2.54;0;0
- K1: JLCPCB_CORRECTION (none) -> 8.89;-3.81;0
- RV1: JLCPCB_CORRECTION (none) -> -2.54;0;180
- U2: JLCPCB_CORRECTION (none) -> 0;0;270
Changed lines of the file:
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@@
+      (effects (font (size 1.27 1.27)) hide)
+    )
+    (property "JLCPCB_CORRECTION" "0;0;270" (id 6) (at 109.22 109.22 0)
       (effects (font (size 1.27 1.27)) hide)
     )
@@
       (effects (font (size 1.27 1.27)) hide)
     )
+    (property "JLCPCB_CORRECTION" "2.54;0;0" (id 5) (at 35.56 31.75 0)
+      (effects (font (size 1.27 1.27)) hide)
+    )
     (pin "1")
     (pin "2")
@@
       (effects (font (size 1.27 1.27)) hide)
     )
+    (property "JLCPCB_CORRECTION" "-2.54;0;180" (id 7) (at 86.36 92.71 0)
+      (effects (font (size 1.27 1.27)) hide)
+    )
     (pin "1")
     (pin "2")
@@
     )
     (property "Comment" "Genuine only" (id 8) (at 214.63 85.09 0)
+      (effects (font (size 1.27 1.27)) hide)
+    )
+    (property "JLCPCB_CORRECTION" "8.89;-3.81;0" (id 9) (at 214.63 85.09 0)
       (effects (font (size 1.27 1.27)) hide)
     )
@@
       (effects (font (size 1.27 1.27)) hide)
     )
+    (property "JLCPCB_CORRECTION" "2.54;0;0" (id 8) (at 22.86 118.11 0)
+      (effects (font (size 1.27 1.27)) hide)
+    )
